File: actuator-board.sch (KiCad schematic (older format))
At the start: 33 parts, among them U1 STM32F302K8U6, U2 MCP1703, U3 MAX3051, X1 16MHz 10ppm

Commit message: Add digikey references for BOM
Parts:
- C10: value 22uF -> 1uF
- C6: digikey# (none) -> 399-17563-1-ND
- C9: digikey# (none) -> 399-11133-1-ND
- CONN1, CONN2, TP1, TP2, TP3, TP4, TP5: DNP (none) -> 1
- CONN3, CONN4: digikey# (none) -> WM7622CT-ND
- D1: Digikey VLMTG1300-GS08CT-ND -> (none); digikey# (none) -> VLMTG1300-GS08CT-ND
- D2: Digikey SBR130S3-7DICT-ND -> (none); digikey# (none) -> SBR130S3-7DICT-ND
- R1: digikey# (none) -> 311-510GRCT-ND
- R4: digikey# (none) -> 311-330HRCT-ND
- U1: Digikey 497-14700-ND -> (none); digikey# (none) -> 497-14700-ND
- U2: Digikey MCP1703T-3302E/CBCT-ND -> (none); digikey# (none) -> MCP1703T-3302E/CBCT-ND
- U3: Digikey MAX3051EKA+TCT-ND -> (none); digikey# (none) -> MAX3051EKA+TCT-ND
- X1: Digikey SER4069CT-ND -> (none); digikey# (none) -> SER4069CT-ND
Changed lines of the file:
@@
 EESchema Schematic File Version 4
-LIBS:actuator-board-cache
 EELAYER 30 0
 EELAYER END
@@
 F 2 "Crystal:Crystal_SMD_SeikoEpson_TSX3225-4Pin_3.2x2.5mm" H 5950 5850 60  0001 C CNN
 F 3 "" H 5950 5850 60  0000 C CNN
-F 4 "SER4069CT-ND" H 5950 6150 60  0000 C CNN "Digikey"
+F 4 "SER4069CT-ND" H 5950 6150 60  0000 C CNN "digikey#"
 	1    5950 5850
 	1    0    0    -1
@@
 F 2 "Connector_Molex:Molex_PicoBlade_53398-0471_1x04-1MP_P1.25mm_Vertical" H 10750 4950 50  0001 C CNN
 F 3 "DOCUMENTATION" H 10750 4950 50  0001 C CNN
+F 4 "WM7622CT-ND" H 10500 4950 50  0001 C CNN "digikey#"
 	1    10500 4950
 	1    0    0    -1
@@
 F 2 "Connector_Molex:Molex_PicoBlade_53398-0471_1x04-1MP_P1.25mm_Vertical" H 10750 5900 50  0001 C CNN
 F 3 "DOCUMENTATION" H 10750 5900 50  0001 C CNN
+F 4 "WM7622CT-ND" H 10500 5900 50  0001 C CNN "digikey#"
 	1    10500 5900
 	1    0    0    -1
@@
 F 2 "_std:_SOT23-8" H 8900 5450 50  0001 C CNN
 F 3 "CAN Transceiver" H 8900 5450 50  0001 C CNN
-F 4 "MAX3051EKA+TCT-ND" H 8850 5900 50  0000 C CNN "Digikey"
+F 4 "MAX3051EKA+TCT-ND" H 8850 5900 50  0001 C CNN "digikey#"
 	1    8900 5450
 	1    0    0    -1
@@
 F 2 "Capacitor_SMD:C_0603_1608Metric" H 5638 5850 50  0001 C CNN
 F 3 "" H 5600 6000 50  0000 C CNN
+F 4 "399-17563-1-ND" H 5600 6000 50  0001 C CNN "digikey#"
 	1    5600 6000
 	1    0    0    -1
@@
 F 2 "Connector_Molex:Molex_PicoBlade_53048-0710_1x07_P1.25mm_Horizontal" H 1400 1750 50  0001 C CNN
 F 3 "DOCUMENTATION" H 1400 1750 50  0001 C CNN
+F 4 "1" H 1400 1800 50  0001 C CNN "DNP"
 	1    1400 1800
 	-1   0    0    -1
@@
 P 9450 1200
 F 0 "C10" H 9475 1300 50  0000 L CNN
-F 1 "22uF" H 9475 1100 50  0000 L CNN
+F 1 "1uF" H 9475 1100 50  0000 L CNN
 F 2 "Capacitor_SMD:C_0603_1608Metric" H 9488 1050 50  0001 C CNN
 F 3 "" H 9450 1200 50  0000 C CNN
@@
 F 2 "_div:_MCP1703-SOT-23A" H 8750 1450 60  0001 C CNN
 F 3 "" H 8750 1450 60  0000 C CNN
-F 4 "MCP1703T-3302E/CBCT-ND" H 8850 1300 50  0000 C CNN "Digikey"
+F 4 "MCP1703T-3302E/CBCT-ND" H 8850 1300 50  0001 C CNN "digikey#"
 	1    8850 1000
 	1    0    0    -1
@@
 F 2 "Capacitor_SMD:C_0603_1608Metric" H 8288 1050 50  0001 C CNN
 F 3 "" H 8250 1200 50  0000 C CNN
+F 4 "399-11133-1-ND" H 8250 1200 50  0001 C CNN "digikey#"
 	1    8250 1200
 	1    0    0    -1
@@
 F 2 "Diode_SMD:D_SOD-323_HandSoldering" V 7800 1000 50  0001 C CNN
 F 3 "~" V 7800 1000 50  0001 C CNN
-F 4 "SBR130S3-7DICT-ND" H 7800 887 50  0000 C CNN "Digikey"
+F 4 "SBR130S3-7DICT-ND" H 7800 887 50  0001 C CNN "digikey#"
 	1    7800 1000
 	-1   0    0    1
@@
 F 2 "Connector_PinHeader_2.54mm:PinHeader_1x02_P2.54mm_Vertical" H 3950 1600 50  0001 C CNN
 F 3 "DOCUMENTATION" H 3950 1600 50  0001 C CNN
+F 4 "1" H 3700 1600 50  0001 C CNN "DNP"
 	1    3700 1600
 	-1   0    0    -1
@@
 F 2 "Package_DFN_QFN:QFN-32-1EP_5x5mm_P0.5mm_EP3.45x3.45mm" H 4600 3950 60  0001 C CNN
 F 3 "DOCUMENTATION" H 4600 3950 60  0001 C CNN
-F 4 "497-14700-ND" H 4450 6100 50  0000 C CNN "Digikey"
+F 4 "497-14700-ND" H 4450 6100 50  0000 C CNN "digikey#"
 	1    4600 4450
 	1    0    0    -1
@@
 F 2 "Resistor_SMD:R_0603_1608Metric" V 1555 4325 50  0001 C CNN
 F 3 "" H 1625 4325 50  0000 C CNN
+F 4 "311-510GRCT-ND" V 1625 4325 50  0001 C CNN "digikey#"
 	1    1625 4325
 	1    0    0    -1
@@
 F 2 "LED_SMD:LED_0603_1608Metric" H 1625 4725 50  0001 C CNN
 F 3 "" H 1625 4725 50  0000 C CNN
-F 4 "VLMTG1300-GS08CT-ND" H 1675 4525 50  0000 C CNN "Digikey"
+F 4 "VLMTG1300-GS08CT-ND" H 1675 4525 50  0000 C CNN "digikey#"
 	1    1625 4725
 	0    -1   -1   0
@@
 F 2 "Resistor_SMD:R_0603_1608Metric" H 5900 4000 50  0001 C CNN
 F 3 "~" H 5900 4000 50  0001 C CNN
+F 4 "311-330HRCT-ND" V 5900 4000 50  0001 C CNN "digikey#"
 	1    5900 4000
 	0    1    1    0
@@
 F 2 "TestPoint:TestPoint_Pad_D1.0mm" H 5700 1600 50  0001 C CNN
 F 3 "~" H 5700 1600 50  0001 C CNN
+F 4 "1" V 5500 1600 50  0001 C CNN "DNP"
 	1    5500 1600
 	0    1    1    0
@@
 F 2 "TestPoint:TestPoint_Pad_D1.0mm" H 5700 1400 50  0001 C CNN
 F 3 "~" H 5700 1400 50  0001 C CNN
+F 4 "1" V 5500 1400 50  0001 C CNN "DNP"
 	1    5500 1400
 	0    1    1    0
@@
 F 2 "TestPoint:TestPoint_Pad_D1.0mm" H 5700 1500 50  0001 C CNN
 F 3 "~" H 5700 1500 50  0001 C CNN
+F 4 "1" V 5500 1500 50  0001 C CNN "DNP"
 	1    5500 1500
 	0    1    1    0
@@
 F 2 "TestPoint:TestPoint_Pad_D1.0mm" H 5700 1700 50  0001 C CNN
 F 3 "~" H 5700 1700 50  0001 C CNN
+F 4 "1" V 5500 1700 50  0001 C CNN "DNP"
 	1    5500 1700
 	0    1    1    0
@@
 F 2 "TestPoint:TestPoint_Pad_D1.0mm" H 5700 1800 50  0001 C CNN
 F 3 "~" H 5700 1800 50  0001 C CNN
+F 4 "1" V 5500 1800 50  0001 C CNN "DNP"
 	1    5500 1800
 	0    1    1    0

Commit message: Update footprints, better refdes, cleanup schematic, 40x22mm outline
Parts:
- removed H1, H2, H3, H4: MountingHole, MountingHole:MountingHole_2.2mm_M2, symbol Mechanical:MountingHole
- J5: renamed from CONN1; footprint Connector_Molex:Molex_PicoBlade_53048-0710_1x07_P1.25mm_Horizontal -> Connector_Molex:Molex_PicoBlade_53047-0710_1x07_P1.25mm_Vertical
- J7: renamed from CONN3; footprint Connector_Molex:Molex_PicoBlade_53398-0471_1x04-1MP_P1.25mm_Vertical -> Connector_Molex:Molex_PicoBlade_53261-0471_1x04-1MP_P1.25mm_Horizontal
- J8: renamed from CONN4; footprint Connector_Molex:Molex_PicoBlade_53398-0471_1x04-1MP_P1.25mm_Vertical -> Connector_Molex:Molex_PicoBlade_53261-0471_1x04-1MP_P1.25mm_Horizontal
- U2: footprint _div:_MCP1703-SOT-23A -> Package_TO_SOT_SMD:SOT-23_Handsoldering
- U3: footprint _std:_SOT23-8 -> Package_TO_SOT_SMD:SOT-23-8
- renumbered CONN2 to J6
Changed lines of the file:
@@
 EESchema Schematic File Version 4
+LIBS:actuator-board-cache
 EELAYER 30 0
 EELAYER END
@@
 $EndComp
 $Comp
-L _connectors:CAN CONN3
+L _connectors:CAN J7
 U 1 1 56D60A8A
 P 10500 4950
-F 0 "CONN3" H 10500 5300 50  0000 C CNN
+F 0 "J7" H 10500 5300 50  0000 C CNN
 F 1 "CAN" H 10500 4600 50  0000 C CNN
-F 2 "Connector_Molex:Molex_PicoBlade_53398-0471_1x04-1MP_P1.25mm_Vertical" H 10750 4950 50  0001 C CNN
+F 2 "Connector_Molex:Molex_PicoBlade_53261-0471_1x04-1MP_P1.25mm_Horizontal" H 10750 4950 50  0001 C CNN
 F 3 "DOCUMENTATION" H 10750 4950 50  0001 C CNN
 F 4 "WM7622CT-ND" H 10500 4950 50  0001 C CNN "digikey#"
@@
 $EndComp
 $Comp
-L _connectors:CAN CONN4
+L _connectors:CAN J8
 U 1 1 56D60AB3
 P 10500 5900
-F 0 "CONN4" H 10500 6250 50  0000 C CNN
+F 0 "J8" H 10500 6250 50  0000 C CNN
 F 1 "CAN" H 10500 5550 50  0000 C CNN
-F 2 "Connector_Molex:Molex_PicoBlade_53398-0471_1x04-1MP_P1.25mm_Vertical" H 10750 5900 50  0001 C CNN
+F 2 "Connector_Molex:Molex_PicoBlade_53261-0471_1x04-1MP_P1.25mm_Horizontal" H 10750 5900 50  0001 C CNN
 F 3 "DOCUMENTATION" H 10750 5900 50  0001 C CNN
 F 4 "WM7622CT-ND" H 10500 5900 50  0001 C CNN "digikey#"
@@
 F 0 "U3" H 9300 5800 50  0000 C CNN
 F 1 "MAX3051" H 8600 5800 50  0000 C CNN
-F 2 "_std:_SOT23-8" H 8900 5450 50  0001 C CNN
+F 2 "Package_TO_SOT_SMD:SOT-23-8" H 8900 5450 50  0001 C CNN
 F 3 "CAN Transceiver" H 8900 5450 50  0001 C CNN
 F 4 "MAX3051EKA+TCT-ND" H 8850 5900 50  0001 C CNN "digikey#"
@@
 UART1TX
 $Comp
-L _connectors:SWD_DEBUG CONN1
+L _connectors:SWD_DEBUG J5
 U 1 1 56D60ADA
 P 1400 1800
-F 0 "CONN1" H 1400 2250 50  0000 C CNN
+F 0 "J5" H 1400 2250 50  0000 C CNN
 F 1 "SWD/DEBUG" H 1400 1350 50  0000 C CNN
-F 2 "Connector_Molex:Molex_PicoBlade_53048-0710_1x07_P1.25mm_Horizontal" H 1400 1750 50  0001 C CNN
+F 2 "Connector_Molex:Molex_PicoBlade_53047-0710_1x07_P1.25mm_Vertical" H 1400 1750 50  0001 C CNN
 F 3 "DOCUMENTATION" H 1400 1750 50  0001 C CNN
 F 4 "1" H 1400 1800 50  0001 C CNN "DNP"
@@
 F 0 "U2" H 9100 1200 60  0000 C CNN
 F 1 "MCP1703" H 8800 1200 60  0000 C CNN
-F 2 "_div:_MCP1703-SOT-23A" H 8750 1450 60  0001 C CNN
+F 2 "Package_TO_SOT_SMD:SOT-23_Handsoldering" H 8750 1450 60  0001 C CNN
 F 3 "" H 8750 1450 60  0000 C CNN
 F 4 "MCP1703T-3302E/CBCT-ND" H 8850 1300 50  0001 C CNN "digikey#"
@@
 VACUUM_SENS_RESET
 $Comp
-L _connectors:PWR CONN2
+L _connectors:PWR J6
 U 1 1 5E236F0F
 P 3700 1600
-F 0 "CONN2" H 3650 1400 50  0000 C CNN
+F 0 "J6" H 3650 1400 50  0000 C CNN
 F 1 "BATTERY" H 3650 1800 50  0000 C CNN
 F 2 "Connector_PinHeader_2.54mm:PinHeader_1x02_P2.54mm_Vertical" H 3950 1600 50  0001 C CNN
@@
 Text Label 5450 3100 0    60   ~ 0
 ANALOG1
-$Comp
-L Mechanical:MountingHole H1
-U 1 1 5E4606C0
-P 3250 6800
-F 0 "H1" H 3350 6846 50  0000 L CNN
-F 1 "MountingHole" H 3350 6755 50  0000 L CNN
-F 2 "MountingHole:MountingHole_2.2mm_M2" H 3250 6800 50  0001 C CNN
-F 3 "~" H 3250 6800 50  0001 C CNN
-	1    3250 6800
-	1    0    0    -1
-$EndComp
-$Comp
-L Mechanical:MountingHole H2
-U 1 1 5E46075F
-P 3250 7000
-F 0 "H2" H 3350 7046 50  0000 L CNN
-F 1 "MountingHole" H 3350 6955 50  0000 L CNN
-F 2 "MountingHole:MountingHole_2.2mm_M2" H 3250 7000 50  0001 C CNN
-F 3 "~" H 3250 7000 50  0001 C CNN
-	1    3250 7000
-	1    0    0    -1
-$EndComp
-$Comp
-L Mechanical:MountingHole H3
-U 1 1 5E460FB2
-P 3250 7200
-F 0 "H3" H 3350 7246 50  0000 L CNN
-F 1 "MountingHole" H 3350 7155 50  0000 L CNN
-F 2 "MountingHole:MountingHole_2.2mm_M2" H 3250 7200 50  0001 C CNN
-F 3 "~" H 3250 7200 50  0001 C CNN
-	1    3250 7200
-	1    0    0    -1
-$EndComp
-$Comp
-L Mechanical:MountingHole H4
-U 1 1 5E4612D7
-P 3250 7400
-F 0 "H4" H 3350 7446 50  0000 L CNN
-F 1 "MountingHole" H 3350 7355 50  0000 L CNN
-F 2 "MountingHole:MountingHole_2.2mm_M2" H 3250 7400 50  0001 C CNN
-F 3 "~" H 3250 7400 50  0001 C CNN
-	1    3250 7400
-	1    0    0    -1
-$EndComp
 $EndSCHEMATC

Commit message: Update authors, DRC rules, layers, track/via settings
Changed lines of the file:
@@
 Rev "A.4"
 Comp "Club Vaudois de Robotique Autonome"
-Comment1 "Salah Missri"
-Comment2 "Authors: Patrick Spieler, Michael Spieler, "
+Comment1 "Michael Spieler, Salah Missri, Antoine Albertelli"
+Comment2 "Authors: "
 Comment3 ""
 Comment4 ""
@@
 F 2 "Crystal:Crystal_SMD_SeikoEpson_TSX3225-4Pin_3.2x2.5mm" H 5950 5850 60  0001 C CNN
 F 3 "" H 5950 5850 60  0000 C CNN
-F 4 "SER4069CT-ND" H 5950 6150 60  0000 C CNN "digikey#"
+F 4 "SER4069CT-ND" H 5950 6150 60  0001 C CNN "digikey#"
 	1    5950 5850
 	1    0    0    -1
@@
 Connection ~ 9450 1000
 Wire Wire Line
-	7250 1000 7700 1000
+	7450 1000 7700 1000
 $Comp
 L Device:D_Schottky_Small D2
 U 1 1 5BD6F803
 P 7800 1000
-F 0 "D2" H 7800 705 50  0000 C CNN
-F 1 "SBR130S3-7" H 7800 796 50  0000 C CNN
+F 0 "D2" H 7800 900 50  0000 C CNN
+F 1 "SBR130S3-7" H 7800 1100 50  0000 C CNN
 F 2 "Diode_SMD:D_SOD-323_HandSoldering" V 7800 1000 50  0001 C CNN
 F 3 "~" V 7800 1000 50  0001 C CNN
@@
 F 2 "Package_DFN_QFN:QFN-32-1EP_5x5mm_P0.5mm_EP3.45x3.45mm" H 4600 3950 60  0001 C CNN
 F 3 "DOCUMENTATION" H 4600 3950 60  0001 C CNN
-F 4 "497-14700-ND" H 4450 6100 50  0000 C CNN "digikey#"
+F 4 "497-14700-ND" H 4450 6100 50  0001 C CNN "digikey#"
 	1    4600 4450
 	1    0    0    -1
@@
 F 2 "LED_SMD:LED_0603_1608Metric" H 1625 4725 50  0001 C CNN
 F 3 "" H 1625 4725 50  0000 C CNN
-F 4 "VLMTG1300-GS08CT-ND" H 1675 4525 50  0000 C CNN "digikey#"
+F 4 "VLMTG1300-GS08CT-ND" H 1675 4525 50  0001 C CNN "digikey#"
 	1    1625 4725
 	0    -1   -1   0
@@
 L power:+5V #PWR0108
 U 1 1 5E459C00
-P 7250 1000
-F 0 "#PWR0108" H 7250 850 50  0001 C CNN
-F 1 "+5V" H 7265 1173 50  0000 C CNN
-F 2 "" H 7250 1000 50  0001 C CNN
-F 3 "" H 7250 1000 50  0001 C CNN
-	1    7250 1000
-	1    0    0    -1
-$EndComp
+P 7450 1000
+F 0 "#PWR0108" H 7450 850 50  0001 C CNN
+F 1 "+5V" H 7465 1173 50  0000 C CNN
+F 2 "" H 7450 1000 50  0001 C CNN
+F 3 "" H 7450 1000 50  0001 C CNN
+	1    7450 1000
+	1    0    0    -1
+$EndComp

Commit message: layout: CAN, rearrange LED/CS1/CS2
Connections:
- net LED: now also U1.15 (PB0); no longer U1.25 (PA15)
- net SPI_CS1: now also U1.18 (PA8); no longer U1.15 (PB0)
- net SPI_CS2: now also U1.25 (PA15); no longer U1.18 (PA8)
Changed lines of the file:
@@
 	1    0    0    -1
 $EndComp
-Text Label 5450 4600 0    60   ~ 0
+Text Label 5450 4850 0    60   ~ 0
 LED
 $Comp
@@
 Text Label 5450 5000 0    60   ~ 0
 SPI_SCK
-Text Label 5450 4850 0    60   ~ 0
+Text Label 5450 3900 0    60   ~ 0
 SPI_CS1
-Text Label 5450 3900 0    60   ~ 0
+Text Label 5450 4600 0    60   ~ 0
 SPI_CS2
 $Comp
