File: Sensors.sch (KiCad schematic (older format))
At the start: 13 parts, among them J2 Conn_01x06, U4 MPRLS0015PA0000SA, U5 MPRLS0015PA0000SA

Commit message: Add digikey references for BOM
Parts:
- C13: digikey# (none) -> 399-8984-1-ND
- J2: digikey# (none) -> WM7612CT-ND
- U4: digikey# (none) -> 480-7099-1-ND
Changed lines of the file:
@@
 EESchema Schematic File Version 4
-LIBS:actuator-board-cache
 EELAYER 30 0
 EELAYER END
@@
 F 2 "_sensors:MPR" H 4200 2900 50  0001 L CNN
 F 3 "https://sensing.honeywell.com/honeywell-sensing-micropressure-board-mount-pressure-mpr-series-datasheet-32332628.pdf" H 4300 2275 50  0001 L CNN
+F 4 "480-7099-1-ND" H 4200 2900 50  0001 C CNN "digikey#"
 	1    4200 2900
 	1    0    0    -1
@@
 F 2 "Capacitor_SMD:C_0603_1608Metric" H 5100 2650 50  0001 C CNN
 F 3 "~" H 5100 2650 50  0001 C CNN
+F 4 "399-8984-1-ND" H 5100 2650 50  0001 C CNN "digikey#"
 	1    5100 2650
 	1    0    0    -1
@@
 F 2 "Connector_Molex:Molex_PicoBlade_53261-0671_1x06-1MP_P1.25mm_Horizontal" H 4550 4750 50  0001 C CNN
 F 3 "~" H 4550 4750 50  0001 C CNN
+F 4 "WM7612CT-ND" H 4550 4750 50  0001 C CNN "digikey#"
 	1    4550 4750
 	1    0    0    -1

Commit message: Update footprints, better refdes, cleanup schematic, 40x22mm outline
Parts:
- U4: footprint _sensors:MPR -> _sensors:MPR-AbsoluteRef
- U5: footprint _sensors:MPR -> _sensors:MPR-AbsoluteRef; digikey# (none) -> 480-7099-1-ND
Changed lines of the file:
@@
 EESchema Schematic File Version 4
+LIBS:actuator-board-cache
 EELAYER 30 0
 EELAYER END
@@
 F 0 "U4" H 3750 3350 50  0000 C CNN
 F 1 "MPRLS0015PA0000SA" H 4650 3350 50  0000 C CNN
-F 2 "_sensors:MPR" H 4200 2900 50  0001 L CNN
+F 2 "_sensors:MPR-AbsoluteRef" H 4200 2900 50  0001 L CNN
 F 3 "https://sensing.honeywell.com/honeywell-sensing-micropressure-board-mount-pressure-mpr-series-datasheet-32332628.pdf" H 4300 2275 50  0001 L CNN
 F 4 "480-7099-1-ND" H 4200 2900 50  0001 C CNN "digikey#"
@@
 F 0 "U5" H 7200 3350 50  0000 C CNN
 F 1 "MPRLS0015PA0000SA" H 8100 3350 50  0000 C CNN
-F 2 "_sensors:MPR" H 7650 2900 50  0001 L CNN
+F 2 "_sensors:MPR-AbsoluteRef" H 7650 2900 50  0001 L CNN
 F 3 "https://sensing.honeywell.com/honeywell-sensing-micropressure-board-mount-pressure-mpr-series-datasheet-32332628.pdf" H 7750 2275 50  0001 L CNN
+F 4 "480-7099-1-ND" H 7650 2900 50  0001 C CNN "digikey#"
 	1    7650 2900
 	1    0    0    -1
@@
 Text Notes 2400 2150 0    60   ~ 0
 Notes:\n- Absolute pressure\n- 0-1 atm\n- SPI mode\n- output range: 24bits 10%-90%
-Text Notes 1000 5000 0    60   ~ 0
+Text Notes 800  4900 0    60   ~ 0
 Input range = 0-6.6V\nFc = 318 Hz\n(10k+10k)/(10k*10k*100nF*2*pi)
 Wire Notes Line
-	2250 5600 2350 5600
+	2500 5350 2600 5350
 Wire Notes Line
-	2350 5600 2350 4400
+	2500 5350 2500 4150
 Wire Notes Line
-	2350 4400 2250 4400
-Text Notes 1450 6250 0    60   ~ 0
+	2600 4150 2500 4150
+Text Notes 3550 6200 0    60   ~ 0
 Input range = 0-3.3V
 $Comp

Commit message: Update DigiKey references
Parts:
- C11, C12, C14, C16: digikey# (none) -> 399-1283-1-ND
- C15: digikey# (none) -> 399-8984-1-ND
- J2: digikey# WM7612CT-ND -> WM7626CT-ND
- R10, R7, R8, R9: digikey# (none) -> 311-10KGRCT-ND
Changed lines of the file:
@@
 F 2 "Capacitor_SMD:C_0603_1608Metric" H 3400 4500 50  0001 C CNN
 F 3 "~" H 3400 4500 50  0001 C CNN
+F 4 "399-1283-1-ND" H 3400 4500 50  0001 C CNN "digikey#"
 	1    3400 4500
 	1    0    0    -1
@@
 F 2 "Resistor_SMD:R_0603_1608Metric" H 3675 5000 50  0001 C CNN
 F 3 "~" H 3675 5000 50  0001 C CNN
+F 4 "311-10KGRCT-ND" H 3675 5000 50  0001 C CNN "digikey#"
 	1    3675 5000
 	1    0    0    -1
@@
 F 2 "Capacitor_SMD:C_0603_1608Metric" H 3400 5300 50  0001 C CNN
 F 3 "~" H 3400 5300 50  0001 C CNN
+F 4 "399-1283-1-ND" H 3400 5300 50  0001 C CNN "digikey#"
 	1    3400 5300
 	1    0    0    -1
@@
 F 2 "Resistor_SMD:R_0603_1608Metric" H 3675 5300 50  0001 C CNN
 F 3 "~" H 3675 5300 50  0001 C CNN
+F 4 "311-10KGRCT-ND" H 3675 5300 50  0001 C CNN "digikey#"
 	1    3675 5300
 	1    0    0    -1
@@
 F 2 "Capacitor_SMD:C_0603_1608Metric" H 5550 2400 50  0001 C CNN
 F 3 "~" H 5550 2400 50  0001 C CNN
+F 4 "399-1283-1-ND" H 5550 2400 50  0001 C CNN "digikey#"
 	1    5550 2400
 	-1   0    0    1
@@
 F 2 "Resistor_SMD:R_0603_1608Metric" H 3650 4200 50  0001 C CNN
 F 3 "~" H 3650 4200 50  0001 C CNN
+F 4 "311-10KGRCT-ND" H 3650 4200 50  0001 C CNN "digikey#"
 	1    3650 4200
 	1    0    0    -1
@@
 F 2 "Resistor_SMD:R_0603_1608Metric" H 3650 4500 50  0001 C CNN
 F 3 "~" H 3650 4500 50  0001 C CNN
+F 4 "311-10KGRCT-ND" H 3650 4500 50  0001 C CNN "digikey#"
 	1    3650 4500
 	1    0    0    -1
@@
 F 2 "Capacitor_SMD:C_0603_1608Metric" H 9000 2400 50  0001 C CNN
 F 3 "~" H 9000 2400 50  0001 C CNN
+F 4 "399-1283-1-ND" H 9000 2400 50  0001 C CNN "digikey#"
 	1    9000 2400
 	-1   0    0    1
@@
 F 2 "Capacitor_SMD:C_0603_1608Metric" H 8550 2650 50  0001 C CNN
 F 3 "~" H 8550 2650 50  0001 C CNN
+F 4 "399-8984-1-ND" H 8550 2650 50  0001 C CNN "digikey#"
 	1    8550 2650
 	1    0    0    -1
@@
 F 2 "Connector_Molex:Molex_PicoBlade_53261-0671_1x06-1MP_P1.25mm_Horizontal" H 4550 4750 50  0001 C CNN
 F 3 "~" H 4550 4750 50  0001 C CNN
-F 4 "WM7612CT-ND" H 4550 4750 50  0001 C CNN "digikey#"
+F 4 "WM7626CT-ND" H 4550 4750 50  0001 C CNN "digikey#"
 	1    4550 4750
 	1    0    0    -1

Commit message: Fixed analog/digital input connector reference
Parts:
- J2: digikey# WM7626CT-ND -> WM7624CT-ND
Changed lines of the file:
@@
 F 2 "Connector_Molex:Molex_PicoBlade_53261-0671_1x06-1MP_P1.25mm_Horizontal" H 4550 4750 50  0001 C CNN
 F 3 "~" H 4550 4750 50  0001 C CNN
-F 4 "WM7626CT-ND" H 4550 4750 50  0001 C CNN "digikey#"
+F 4 "WM7624CT-ND" H 4550 4750 50  0001 C CNN "digikey#"
 	1    4550 4750
 	1    0    0    -1
